Commit message: [modify] calibrated kinect left

File: motoman_description/robots/sia5/sia5_with_dhand_and_3_kinects.urdf.xacro (robot description, xacro)
@@ -47,5 +47,6 @@
   <joint name="joint_left_right" type="fixed">
   <!-- Calibrated position -->
-  <origin xyz="-0.513 1.0085 0.756" rpy="0.0126 0.2924 -0.634" />
+  <!-- <origin xyz="-0.513 1.0085 0.756" rpy="0.0126 0.2924 -0.634" /> -->
+  <origin xyz="-0.513925 0.995299 0.72318" rpy="3.14041 2.90483 2.50322" />
   <!-- Test positions -->
   <!-- <origin xyz="-0.600 0.800 0.600" rpy="-0.01 0.3206 -0.4815" /> -->

Commit message: [modify] chenged the position of kinect_left

File: motoman_description/robots/sia5/sia5_with_dhand_and_3_kinects.urdf.xacro (robot description, xacro)
@@ -46,7 +46,10 @@
   <!-- Joint -->
   <joint name="joint_left_right" type="fixed">
+  <!-- Original position -->
+  <origin xyz="-0.513 1.0085 0.756" rpy="0.0126 0.2924 -0.634" />
   <!-- Calibrated position -->
-  <!-- <origin xyz="-0.513 1.0085 0.756" rpy="0.0126 0.2924 -0.634" /> -->
-  <origin xyz="-0.513925 0.995299 0.72318" rpy="3.14041 2.90483 2.50322" />
+  <!-- <origin xyz="-0.513925 0.995299 0.72318" rpy="3.14041 2.90483 2.50322" /> -->
+  <!-- Calibrated by InteractiveMarker 2018/7/31 -->
+  <!-- <origin xyz="-0.5321 0.9764 0.7601" rpy="0.012 0.2605 -0.6153" /> -->
   <!-- Test positions -->
   <!-- <origin xyz="-0.600 0.800 0.600" rpy="-0.01 0.3206 -0.4815" /> -->
